Commit message: nicola: bugfix

File: cnr_ros_control_test_description/urdf/ur10.urdf.xacro (robot description, xacro)
@@ -27,5 +27,5 @@
     safety_k_position:=20
     kinematics_file">
-    <xacro:property name="__kinematics" value="${kinematics_file['kinematics']}"/>
+    <xacro:property name="f_kinematics" value="${kinematics_file['kinematics']}"/>
     <!-- Inertia parameters -->
     <xacro:property name="base_mass" value="4.0" />  <!-- This mass might be incorrect -->
@@ -75,5 +75,5 @@
       <parent link="${prefix}base_link" />
       <child link = "${prefix}shoulder_link" />
-      <origin xyz="${__kinematics['shoulder']['x']} ${__kinematics['shoulder']['y']} ${__kinematics['shoulder']['z']}" rpy="${__kinematics['shoulder']['roll']} ${__kinematics['shoulder']['pitch']} ${__kinematics['shoulder']['yaw'] + base_correction}" />
+      <origin xyz="${f_kinematics['shoulder']['x']} ${f_kinematics['shoulder']['y']} ${f_kinematics['shoulder']['z']}" rpy="${f_kinematics['shoulder']['roll']} ${f_kinematics['shoulder']['pitch']} ${f_kinematics['shoulder']['yaw'] + base_correction}" />
       <axis xyz="0 0 1" />
       <xacro:unless value="${joint_limited}">
@@ -114,5 +114,5 @@
       <parent link="${prefix}shoulder_link" />
       <child link = "${prefix}upper_arm_link" />
-      <origin xyz="${__kinematics['upper_arm']['x']} ${__kinematics['upper_arm']['y']} ${__kinematics['upper_arm']['z']}" rpy="${__kinematics['upper_arm']['roll']} ${__kinematics['upper_arm']['pitch']} ${__kinematics['upper_arm']['yaw']}" />
+      <origin xyz="${f_kinematics['upper_arm']['x']} ${f_kinematics['upper_arm']['y']} ${f_kinematics['upper_arm']['z']}" rpy="${f_kinematics['upper_arm']['roll']} ${f_kinematics['upper_arm']['pitch']} ${f_kinematics['upper_arm']['yaw']}" />
       <axis xyz="0 0 1" />
       <xacro:unless value="${joint_limited}">
@@ -146,6 +146,6 @@
         </geometry>
       </collision>
-      <xacro:cylinder_inertial radius="0.075" length="${-1*__kinematics['forearm']['x']}" mass="${upper_arm_mass}">
-        <origin xyz="${0.5*__kinematics['forearm']['x']} 0.0 ${upper_arm_inertia_offset}" rpy="0 ${pi/2} 0" />
+      <xacro:cylinder_inertial radius="0.075" length="${-1*f_kinematics['forearm']['x']}" mass="${upper_arm_mass}">
+        <origin xyz="${0.5*f_kinematics['forearm']['x']} 0.0 ${upper_arm_inertia_offset}" rpy="0 ${pi/2} 0" />
       </xacro:cylinder_inertial>
     </link>
@@ -153,5 +153,5 @@
       <parent link="${prefix}upper_arm_link" />
       <child link = "${prefix}forearm_link" />
-      <origin xyz="${__kinematics['forearm']['x']} ${__kinematics['forearm']['y']} ${__kinematics['forearm']['z']}" rpy="${__kinematics['forearm']['roll']} ${__kinematics['forearm']['pitch']} ${__kinematics['forearm']['yaw']}" />
+      <origin xyz="${f_kinematics['forearm']['x']} ${f_kinematics['forearm']['y']} ${f_kinematics['forearm']['z']}" rpy="${f_kinematics['forearm']['roll']} ${f_kinematics['forearm']['pitch']} ${f_kinematics['forearm']['yaw']}" />
       <axis xyz="0 0 1" />
       <xacro:unless value="${joint_limited}">
@@ -185,6 +185,6 @@
         </geometry>
       </collision>
-      <xacro:cylinder_inertial radius="0.075" length="${-1*__kinematics['wrist_1']['x']}" mass="${forearm_mass}">
-        <origin xyz="${0.5*__kinematics['forearm']['x']} 0.0 ${elbow_offset}" rpy="0 ${pi/2} 0" />
+      <xacro:cylinder_inertial radius="0.075" length="${-1*f_kinematics['wrist_1']['x']}" mass="${forearm_mass}">
+        <origin xyz="${0.5*f_kinematics['forearm']['x']} 0.0 ${elbow_offset}" rpy="0 ${pi/2} 0" />
       </xacro:cylinder_inertial>
     </link>
@@ -192,5 +192,5 @@
       <parent link="${prefix}forearm_link" />
       <child link = "${prefix}wrist_1_link" />
-      <origin xyz="${__kinematics['wrist_1']['x']} ${__kinematics['wrist_1']['y']} ${__kinematics['wrist_1']['z']}" rpy="${__kinematics['wrist_1']['roll']} ${__kinematics['wrist_1']['pitch']} ${__kinematics['wrist_1']['yaw']}" />
+      <origin xyz="${f_kinematics['wrist_1']['x']} ${f_kinematics['wrist_1']['y']} ${f_kinematics['wrist_1']['z']}" rpy="${f_kinematics['wrist_1']['roll']} ${f_kinematics['wrist_1']['pitch']} ${f_kinematics['wrist_1']['yaw']}" />
       <axis xyz="0 0 1" />
       <xacro:unless value="${joint_limited}">
@@ -224,5 +224,5 @@
         </geometry>
       </collision>
-      <xacro:cylinder_inertial radius="0.075" length="${-1*__kinematics['wrist_2']['y']}" mass="${wrist_1_mass}">
+      <xacro:cylinder_inertial radius="0.075" length="${-1*f_kinematics['wrist_2']['y']}" mass="${wrist_1_mass}">
         <origin xyz="0.0 0.0 0.0" rpy="0 0 0" />
       </xacro:cylinder_inertial>
@@ -231,5 +231,5 @@
       <parent link="${prefix}wrist_1_link" />
       <child link = "${prefix}wrist_2_link" />
-      <origin xyz="${__kinematics['wrist_2']['x']} ${__kinematics['wrist_2']['y']} ${__kinematics['wrist_2']['z']}" rpy="${__kinematics['wrist_2']['roll']} ${__kinematics['wrist_2']['pitch']} ${__kinematics['wrist_2']['yaw']}" />
+      <origin xyz="${f_kinematics['wrist_2']['x']} ${f_kinematics['wrist_2']['y']} ${f_kinematics['wrist_2']['z']}" rpy="${f_kinematics['wrist_2']['roll']} ${f_kinematics['wrist_2']['pitch']} ${f_kinematics['wrist_2']['yaw']}" />
       <axis xyz="0 0 1" />
       <xacro:unless value="${joint_limited}">
@@ -263,5 +263,5 @@
         </geometry>
       </collision>
-      <xacro:cylinder_inertial radius="0.075" length="${__kinematics['wrist_3']['y']}" mass="${wrist_2_mass}">
+      <xacro:cylinder_inertial radius="0.075" length="${f_kinematics['wrist_3']['y']}" mass="${wrist_2_mass}">
         <origin xyz="0.0 0.0 0.0" rpy="0 0 0" />
       </xacro:cylinder_inertial>
@@ -270,5 +270,5 @@
       <parent link="${prefix}wrist_2_link" />
       <child link = "${prefix}wrist_3_link" />
-      <origin xyz="${__kinematics['wrist_3']['x']} ${__kinematics['wrist_3']['y']} ${__kinematics['wrist_3']['z']}" rpy="${__kinematics['wrist_3']['roll']} ${__kinematics['wrist_3']['pitch']} ${__kinematics['wrist_3']['yaw']}" />
+      <origin xyz="${f_kinematics['wrist_3']['x']} ${f_kinematics['wrist_3']['y']} ${f_kinematics['wrist_3']['z']}" rpy="${f_kinematics['wrist_3']['roll']} ${f_kinematics['wrist_3']['pitch']} ${f_kinematics['wrist_3']['yaw']}" />
       <axis xyz="0 0 1" />
       <xacro:unless value="${joint_limited}">
